Commit message: Adds support for version 2 of the bot(drawers only)

File: dev_ws/src/office_bot_model/models/officebot/robot.urdf (robot description, URDF)
Before this commit: robot onshape, 12 links, 11 joints
Links:
- removed link body
- removed link drawer_1
- removed link drawer_5
- removed link top
- removed link wheel_4
- removed link wheel_4_2
- removed link wheel_4_3
- removed link wheel_4_4
- added link base, mass 15.348841199999997187; collision mesh filename=file:///opt/officebot/models/officebot/base.stl; visual mesh filename=file:///opt/officebot/models/officebot/base.stl
- added link drawer1, mass 1.3157567401165588539; collision mesh filename=file:///opt/officebot/models/officebot/drawer.stl; visual mesh filename=file:///opt/officebot/models/officebot/drawer.stl
- added link lidar, mass 0.14361062151864467662; collision mesh filename=file:///opt/officebot/models/officebot/lidar.stl; visual mesh filename=file:///opt/officebot/models/officebot/lidar.stl
- added link wheel_bl, mass 0.021505374555847410478; collision mesh filename=file:///opt/officebot/models/officebot/wheel.stl; visual mesh filename=file:///opt/officebot/models/officebot/wheel.stl
- added link wheel_br, mass 0.021505374555847410478; collision mesh filename=file:///opt/officebot/models/officebot/wheel.stl; visual mesh filename=file:///opt/officebot/models/officebot/wheel.stl
- added link wheel_tl, mass 0.021505374555847410478; collision mesh filename=file:///opt/officebot/models/officebot/wheel.stl; visual mesh filename=file:///opt/officebot/models/officebot/wheel.stl
- added link wheel_tr, mass 0.021505374555847410478; collision mesh filename=file:///opt/officebot/models/officebot/wheel.stl; visual mesh filename=file:///opt/officebot/models/officebot/wheel.stl
- link drawer_2: mass 12.15096412314713703 -> 1.3157567401165588539; geometry collision mesh filename=file:///opt/officebot/models/officebot/drawer.stl; visual mesh filename=file:///opt/officebot/models/officebot/drawer.stl
- link drawer_3: mass 12.150964123147144136 -> 1.3157567401165588539; geometry collision mesh filename=file:///opt/officebot/models/officebot/drawer.stl; visual mesh filename=file:///opt/officebot/models/officebot/drawer.stl
- link drawer_4: mass 12.150964123147142359 -> 1.3157567401165588539; geometry collision mesh filename=file:///opt/officebot/models/officebot/drawer.stl; visual mesh filename=file:///opt/officebot/models/officebot/drawer.stl
Joints:
- removed joint body_drawer1
- removed joint body_drawer2
- removed joint body_drawer3
- removed joint body_drawer4
- removed joint body_drawer5
- removed joint body_top
- removed joint body_wheel1
- removed joint body_wheel2
- removed joint body_wheel3
- removed joint body_wheel4
- added joint base_drawer1: type prismatic, parent base, child drawer1, origin xyz=0.11500980138576723244 -0.20500000000000001554 0.56999968326568606347 rpy=-1.570796326794896558 -0 3.141592653589793116, axis 0 0 1, limit lower=0 upper=0.4 effort=10 velocity=10
- added joint base_drawer2: type prismatic, parent base, child drawer_2, origin xyz=0.11500980138576727407 -0.20500000000000001554 0.46999968326568986043 rpy=-1.570796326794896558 -0 3.141592653589793116, axis 0 0 1, limit lower=0 upper=0.4 effort=10 velocity=10
- added joint base_drawer3: type prismatic, parent base, child drawer_3, origin xyz=0.11500980138576721856 -0.20500000000000001554 0.36999968326568610788 rpy=-1.570796326794896558 -0 3.141592653589793116, axis 0 0 1, limit lower=0 upper=0.4 effort=10 velocity=10
- added joint base_drawer4: type prismatic, parent base, child drawer_4, origin xyz=0.11500980138576723244 -0.20500000000000001554 0.26999968326568613008 rpy=-1.570796326794896558 -0 3.141592653589793116, axis 0 0 1, limit lower=0 upper=0.4 effort=10 velocity=10
- added joint base_lidar: type revolute, parent base, child lidar, origin xyz=1.561251128379126385e-17 -6.9388939039072283776e-18 0.64000000000000001332 rpy=3.141592653589793116 -0 0, axis 0 0 1, limit lower=0.0 upper=0.35 effort=10 velocity=20
- added joint base_wheel_bl: type revolute, parent base, child wheel_bl, origin xyz=0.13999999999999998557 0.1807999999999999885 -0.025000000000000001388 rpy=-1.570796326794896558 -0 1.570796326794896558, axis 0 0 1, limit effort=10 velocity=20
- added joint base_wheel_br: type revolute, parent base, child wheel_br, origin xyz=-0.14000000000000001332 0.18080000000000001625 -0.025000000000000018735 rpy=3.141592653589793116 -1.570796326794896558 0, axis 0 0 1, limit effort=10 velocity=20
- added joint base_wheel_tl: type revolute, parent base, child wheel_tl, origin xyz=0.14000000000000001332 -0.18080000000000001625 -0.025000000000000001388 rpy=-1.570796326794896558 -0 1.570796326794896558, axis 0 0 1, limit effort=10 velocity=20
- added joint base_wheel_tr: type revolute, parent base, child wheel_tr, origin xyz=-0.14000000000000001332 -0.18080000000000001625 -0.025000000000000011796 rpy=6.7696525891777836328e-17 1.570796326794896558 0, axis 0 0 1, limit effort=10 velocity=20
- joint dummy_root: child body -> base

Commit message: Adds temp support for mecanum wheels

File: dev_ws/src/office_bot_model/models/officebot/robot.urdf (robot description, URDF)
Before this commit: robot officebot, 11 links, 10 joints
Links:
- removed link wheel_bl
- removed link wheel_br
- removed link wheel_tl
- removed link wheel_tr
- added link wheel_fl, mass 0.021505374555847410478; collision sphere radius=0.025; visual mesh filename=file:///opt/officebot/models/officebot/wheel.stl
- added link wheel_fr, mass 0.021505374555847410478; collision sphere radius=0.025; visual mesh filename=file:///opt/officebot/models/officebot/wheel.stl
- added link wheel_rl, mass 0.021505374555847410478; collision sphere radius=0.025; visual mesh filename=file:///opt/officebot/models/officebot/wheel.stl
- added link wheel_rr, mass 0.021505374555847410478; collision sphere radius=0.025; visual mesh filename=file:///opt/officebot/models/officebot/wheel.stl
- link base: mass 15.348841199999997187 -> 5
- link drawer1: mass 1.3157567401165588539 -> 0.5
- link drawer_2: mass 1.3157567401165588539 -> 0.5
- link drawer_3: mass 1.3157567401165588539 -> 0.5
- link drawer_4: mass 1.3157567401165588539 -> 0.5
Joints:
- removed joint base_wheel_bl
- removed joint base_wheel_br
- removed joint base_wheel_tl
- removed joint base_wheel_tr
- added joint base_wheel_fl: type continuous, parent base, child wheel_fl, origin xyz=0.14000000000000001332 -0.18080000000000001625 -0.025000000000000001388 rpy=-1.570796326794896558 -0 1.570796326794896558, axis 0 0 1
- added joint base_wheel_fr: type continuous, parent base, child wheel_fr, origin xyz=-0.14000000000000001332 -0.18080000000000001625 -0.025000000000000011796 rpy=6.7696525891777836328e-17 1.570796326794896558 0, axis 0 0 1
- added joint base_wheel_rl: type continuous, parent base, child wheel_rl, origin xyz=0.13999999999999998557 0.1807999999999999885 -0.025000000000000001388 rpy=-1.570796326794896558 -0 1.570796326794896558, axis 0 0 1
- added joint base_wheel_rr: type continuous, parent base, child wheel_rr, origin xyz=-0.14000000000000001332 0.18080000000000001625 -0.025000000000000018735 rpy=3.141592653589793116 -1.570796326794896558 0, axis 0 0 1

Commit message: Adds support for lidar and imu sensors

File: dev_ws/src/office_bot_model/models/officebot/robot.urdf (robot description, URDF)
Before this commit: robot officebot, 11 links, 10 joints
Joints:
- joint base_lidar: type revolute -> fixed

Commit message: Adds support for lidar and office_world

File: dev_ws/src/office_bot_model/models/officebot/robot.urdf (robot description, URDF)
Before this commit: robot officebot, 11 links, 10 joints
Links:
- removed link lidar
- added link lidar_link, mass 0.14361062151864467662; collision mesh filename=file:///opt/officebot/models/officebot/lidar.stl; visual mesh filename=file:///opt/officebot/models/officebot/lidar.stl
Joints:
- joint base_lidar: child lidar -> lidar_link

Commit message: Adds update for slam toolbox bringup

File: dev_ws/src/office_bot_model/models/officebot/robot.urdf (robot description, URDF)
Before this commit: robot officebot, 11 links, 10 joints
Links:
- removed link dummy_root_link
- added link base_footprint
Joints:
- joint dummy_root: parent dummy_root_link -> base_footprint

Commit message: Removes the bug where wheels move in wrong direction(strafe broken)

File: dev_ws/src/office_bot_model/models/officebot/robot.urdf (robot description, URDF)
Before this commit: robot officebot, 11 links, 10 joints
Joints:
- joint base_lidar: limit lower=0.0 upper=0.35 effort=10 velocity=20 -> (none); parent base -> base_footprint
- joint base_wheel_fl: axis 0 0 1 -> 0 0 -1
- joint base_wheel_rl: axis 0 0 1 -> 0 0 -1

Commit message: fixes problem that caused lidar to move in rviz2

File: dev_ws/src/office_bot_model/models/officebot/robot.urdf (robot description, URDF)
Before this commit: robot office_bot, 11 links, 10 joints
Joints:
- joint base_lidar: parent base_footprint -> base
- joint dummy_root: origin xyz=0 0 0 rpy=0 0 0 -> xyz=0 0 0 rpy=0 0 1.57

Commit message: Adds camera support

File: dev_ws/src/office_bot_model/models/officebot/robot.urdf (robot description, URDF)
Before this commit: robot office_bot, 11 links, 10 joints
Links:
- removed link drawer1
- added link camera_link; visual box size=0.030 0.003 0.03
- added link camera_link_optical
Joints:
- removed joint base_drawer1
- added joint camera_joint: type fixed, parent base, child camera_link, origin xyz=1.561251128379126385e-17 -0.21 0.62000000000000001332 rpy=3.141592653589793116 -0 0, axis 0 0 1
- added joint camera_optical_joint: type fixed, parent camera_link, child camera_link_optical, origin xyz=0 0 0 rpy=3.14 0 1.57

Commit message: new bring up

File: dev_ws/src/office_bot_model/models/officebot/robot.urdf (robot description, URDF)
Before this commit: robot office_bot, 12 links, 11 joints
Links:
- added link drawer_1, mass 1.3157567401165588539; collision mesh filename=package://office_bot_model/models/officebot/drawer.stl; visual mesh filename=package://office_bot_model/models/officebot/drawer.stl
- link base: mass 5 -> 15.49143394549887276; geometry collision mesh filename=package://office_bot_model/models/officebot/91292a073_18_8_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; collision mesh filename=package://office_bot_model/models/officebot/91292a073_18_8_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
- link camera_link: geometry 
- link drawer_2: mass 0.5 -> 1.3157567401165588539; geometry collision mesh filename=package://office_bot_model/models/officebot/drawer.stl; visual mesh filename=package://office_bot_model/models/officebot/drawer.stl
- link drawer_3: mass 0.5 -> 1.3157567401165588539; geometry collision mesh filename=package://office_bot_model/models/officebot/drawer.stl; visual mesh filename=package://office_bot_model/models/officebot/drawer.stl
- link drawer_4: mass 0.5 -> 1.3157567401165588539; geometry collision mesh filename=package://office_bot_model/models/officebot/drawer.stl; visual mesh filename=package://office_bot_model/models/officebot/drawer.stl
- link lidar_link: mass 0.14361062151864467662 -> None; geometry 
- link wheel_fl: geometry collision sphere radius=0.025; visual mesh filename=package://office_bot_model/models/officebot/wheel.stl
- link wheel_fr: geometry collision sphere radius=0.025; visual mesh filename=package://office_bot_model/models/officebot/wheel.stl
- link wheel_rl: geometry collision sphere radius=0.025; visual mesh filename=package://office_bot_model/models/officebot/wheel.stl
- link wheel_rr: geometry collision sphere radius=0.025; visual mesh filename=package://office_bot_model/models/officebot/wheel.stl
Joints:
- added joint base_drawer1: type prismatic, parent base, child drawer_1, origin xyz=0.11500980138576723244 -0.20500000000000001554 0.56999968326568606347 rpy=-1.570796326794896558 -0 3.141592653589793116, axis 0 0 1, limit lower=0 upper=0.4 effort=10 velocity=10
- joint base_lidar: origin xyz=1.561251128379126385e-17 -6.9388939039072283776e-18 0.64000000000000001332 rpy=3.141592653589793116 -0 0 -> xyz=-0.0076784611388689208433 -0.014607735477295019644 0.70535953015098928898 rpy=0 0 0
- joint camera_joint: origin xyz=1.561251128379126385e-17 -0.21 0.62000000000000001332 rpy=3.141592653589793116 -0 0 -> xyz=0.088000000000000008771 -0.16320000000000001172 0.66200000000000003286 rpy=3.141592653589793116 0 0

Commit message: Refactor Officebot model into xacro and stabilize simulation (#4)
- integrate the new Officebot CAD assets into the ROS model package
- make officebot_xacro/main.xacro the canonical robot description
- generate Gazebo-safe robot descriptions with absolute mesh paths at launch time
- preserve camera, lidar, mecanum drive, Nav2, SLAM, and RViz interfaces
- fix drawers as static links and remove the drawer position controller path
- smooth stamped cmd_vel publishing for the mecanum controller
- correct wheel/base geometry and wheel velocity limits for RViz/Gazebo motion
- clean stale RViz fixed-frame configuration

File: dev_ws/src/office_bot_model/models/officebot/robot.urdf (robot description, URDF)
Before this commit: robot office_bot, 12 links, 11 joints
Links:
- added link drawer_1, mass 1.3157567401165588539; collision mesh filename=package://office_bot_model/models/officebot/drawer.stl; visual mesh filename=package://office_bot_model/models/officebot/drawer.stl
- link base: mass 5 -> 15.49143394549887276; geometry collision mesh filename=package://office_bot_model/models/officebot/91292a073_18_8_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; collision mesh filename=package://office_bot_model/models/officebot/91292a073_18_8_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
- link camera_link: geometry 
- link drawer_2: mass 0.5 -> 1.3157567401165588539; geometry collision mesh filename=package://office_bot_model/models/officebot/drawer.stl; visual mesh filename=package://office_bot_model/models/officebot/drawer.stl
- link drawer_3: mass 0.5 -> 1.3157567401165588539; geometry collision mesh filename=package://office_bot_model/models/officebot/drawer.stl; visual mesh filename=package://office_bot_model/models/officebot/drawer.stl
- link drawer_4: mass 0.5 -> 1.3157567401165588539; geometry collision mesh filename=package://office_bot_model/models/officebot/drawer.stl; visual mesh filename=package://office_bot_model/models/officebot/drawer.stl
- link lidar_link: mass 0.14361062151864467662 -> None; geometry 
- link wheel_fl: geometry collision sphere radius=0.025; visual mesh filename=package://office_bot_model/models/officebot/wheel.stl
- link wheel_fr: geometry collision sphere radius=0.025; visual mesh filename=package://office_bot_model/models/officebot/wheel.stl
- link wheel_rl: geometry collision sphere radius=0.025; visual mesh filename=package://office_bot_model/models/officebot/wheel.stl
- link wheel_rr: geometry collision sphere radius=0.025; visual mesh filename=package://office_bot_model/models/officebot/wheel.stl
Joints:
- added joint base_drawer1: type fixed, parent base, child drawer_1, origin xyz=0.11500980138576723244 -0.20500000000000001554 0.5699996832656861 rpy=-1.570796326794896558 0 3.141592653589793116
- joint base_drawer2: axis 0 0 1 -> (none); limit lower=0 upper=0.4 effort=10 velocity=10 -> (none); origin xyz=0.11500980138576727407 -0.20500000000000001554 0.46999968326568986043 rpy=-1.570796326794896558 -0 3.141592653589793116 -> xyz=0.11500980138576723244 -0.20500000000000001554 0.46999968326568986 rpy=-1.570796326794896558 0 3.141592653589793116; type prismatic -> fixed
- joint base_drawer3: axis 0 0 1 -> (none); limit lower=0 upper=0.4 effort=10 velocity=10 -> (none); origin xyz=0.11500980138576721856 -0.20500000000000001554 0.36999968326568610788 rpy=-1.570796326794896558 -0 3.141592653589793116 -> xyz=0.11500980138576723244 -0.20500000000000001554 0.3699996832656861 rpy=-1.570796326794896558 0 3.141592653589793116; type prismatic -> fixed
- joint base_drawer4: axis 0 0 1 -> (none); limit lower=0 upper=0.4 effort=10 velocity=10 -> (none); origin xyz=0.11500980138576723244 -0.20500000000000001554 0.26999968326568613008 rpy=-1.570796326794896558 -0 3.141592653589793116 -> xyz=0.11500980138576723244 -0.20500000000000001554 0.26999968326568613 rpy=-1.570796326794896558 0 3.141592653589793116; type prismatic -> fixed
- joint base_lidar: origin xyz=1.561251128379126385e-17 -6.9388939039072283776e-18 0.64000000000000001332 rpy=3.141592653589793116 -0 0 -> xyz=-0.0076784611388689208433 -0.014607735477295019644 0.70535953015098928898 rpy=0 0 0
- joint camera_joint: origin xyz=1.561251128379126385e-17 -0.21 0.62000000000000001332 rpy=3.141592653589793116 -0 0 -> xyz=0.088000000000000008771 -0.16320000000000001172 0.66200000000000003286 rpy=3.141592653589793116 0 0
- joint dummy_root: origin xyz=0 0 0 rpy=0 0 1.57 -> xyz=0 0 0.05 rpy=0 0 1.57

Commit message: feat: add object-aware detection and navigation workflow
- split object detection into model, localization, tracking, navigation, and web UI modules
- localize detections with projected lidar/scan data and reject stale sensor-frame pairs
- add persistent object tracks with snapshots, duplicate merging, and web-based object selection
- publish detected object obstacle clouds for Nav2 costmaps
- add reachable approach-goal planning, line-of-sight success validation, and no-recovery Nav2 behavior tree
- update Nav2 costmaps, planner settings, camera frames, and package install data

Verification:
- PYTHONPATH=src/object_detector python3 -m pytest src/object_detector/test/test_detector_logic.py
- colcon build --symlink-install --packages-select object_detector

File: dev_ws/src/office_bot_model/models/officebot/robot.urdf (robot description, URDF)
Before this commit: robot office_bot, 13 links, 12 joints
Links:
- added link camera_sensor_link
Joints:
- added joint camera_sensor_joint: type fixed, parent camera_link, child camera_sensor_link, origin xyz=0 0 0 rpy=3.14 0 1.57
- joint camera_optical_joint: origin xyz=0 0 0 rpy=3.14 0 1.57 -> xyz=0 0 0 rpy=-1.5707963267948966 0 -1.5707963267948966; parent camera_link -> camera_sensor_link

File: dev_ws/src/office_bot_model/models/officebot_xacro/sensors.xacro (robot description, xacro)
@@ -16,11 +16,17 @@
             <axis xyz="0 0 1"></axis>
         </joint>
+        <link name="camera_sensor_link"></link>
+        <joint name="camera_sensor_joint" type="fixed">
+            <origin xyz="0 0 0" rpy="3.14 0 1.57"></origin>
+            <parent link="camera_link"></parent>
+            <child link="camera_sensor_link"></child>
+        </joint>
         <link name="camera_link_optical"></link>
         <joint name="camera_optical_joint" type="fixed">
-            <origin xyz="0 0 0" rpy="3.14 0 1.57"></origin>
-            <parent link="camera_link"></parent>
+            <origin xyz="0 0 0" rpy="-1.5707963267948966 0 -1.5707963267948966"></origin>
+            <parent link="camera_sensor_link"></parent>
             <child link="camera_link_optical"></child>
         </joint>
-        <gazebo reference="camera_link_optical">
+        <gazebo reference="camera_sensor_link">
             <sensor name="camera" type="camera">
                 <always_on>true</always_on>
